Commit message: Formatting existing files

File: content/assets/urdf/mug/movable_mug.urdf (robot description, URDF)
Before this commit: robot mug, 7 links, 6 joints
Links:
- removed link base
- removed link base1
- removed link base2
- removed link base3
- removed link base4
- removed link base5
- added link rx
- added link ry
- added link rz
- added link tx
- added link ty
- added link tz
Joints:
- joint rx_joint: child base4 -> ry; parent base3 -> rx
- joint ry_joint: child base5 -> rz; parent base4 -> ry
- joint rz_joint: parent base5 -> rz
- joint x_joint: child base1 -> ty; limit lower=-2 upper=2.0 effort=1 velocity=1 -> lower=-2 upper=2.0 effort=1 velocity=0.1; parent base -> tx
- joint y_joint: child base2 -> tz; limit lower=-2.0 upper=2.0 effort=1 velocity=1 -> lower=-2.0 upper=2.0 effort=1 velocity=0.1; parent base1 -> ty
- joint z_joint: child base3 -> rx; limit lower=-2.8973 upper=2.8973 effort=12 velocity=2.6100 -> lower=-2.8973 upper=2.8973 effort=1 velocity=0.1; parent base2 -> tz
